File: iisi-riser-board.kicad_sch (KiCad schematic)
At the start: 47 parts, among them J1 Conn_01x10_Pin, Q1 DTA114E, Q2 DTC124X, Q3 2SC2412K, Q4 2SC2412K, U1 M51977FP, U2 M51944BML

Commit message: Add Digi-Key part numbers for everything that is brand new
Parts:
- C1: Digi-Key Part (none) -> 399-C0805C331J5GACTUCT-ND
- C10: Digi-Key Part (none) -> 493-3967-1-ND
- C2, C3, C6: Digi-Key Part (none) -> 399-C0805C103K5RACTUCT-ND
- C4: Digi-Key Part (none) -> 445-2283-1-ND
- C5: Digi-Key Part (none) -> 311-1119-1-ND
- C7: Digi-Key Part (none) -> 399-C0805C332J5GACTUCT-ND
- C8: Digi-Key Part (none) -> 399-C0805C102J5GACTUCT-ND
- C9: Digi-Key Part (none) -> 565-4768-1-ND
- D1: Digi-Key Part (none) -> MMBZ5248B-FDICT-ND
- D2: Digi-Key Part (none) -> BZX84C13-FDICT-ND
- D3: Digi-Key Part (none) -> SZBZX84C5V1LT3GOSCT-ND
- D4, D5: Digi-Key Part (none) -> 1727-2887-1-ND
- D6: Digi-Key Part (none) -> SB05-05C-TB-EOSCT-ND
- J1: Digi-Key Part (none) -> A122175CT-ND
- Q1: Digi-Key Part (none) -> DTA114EKAT146CT-ND
- Q2: Digi-Key Part (none) -> DTC124XKAT146CT-ND
- Q3, Q4: Digi-Key Part (none) -> 2SC2412KT146RCT-ND
- R1, R2: Digi-Key Part (none) -> A129765CT-ND
- R10: Digi-Key Part (none) -> A129741CT-ND
- R11: Digi-Key Part (none) -> A127026CT-ND
- R12: Digi-Key Part (none) -> P150KACT-ND
- R13, R15, R17, R3, R6: Digi-Key Part (none) -> A129761CT-ND
- R14: Digi-Key Part (none) -> P33KDACT-ND
- R16, R4: Digi-Key Part (none) -> A129757CT-ND
- R18: Digi-Key Part (none) -> 311-47KARCT-ND
- R19, R20, R21, R22: Digi-Key Part (none) -> P0.0ACT-ND
- R5: Digi-Key Part (none) -> P100DACT-ND
- R7: Digi-Key Part (none) -> A129749CT-ND
- R8: Digi-Key Part (none) -> A129773CT-ND
- R9: Digi-Key Part (none) -> 13-RC0805FR-078R2LCT-ND
- RV1: Digi-Key Part (none) -> 118-TC33X-1-222ECT-ND
